File: ESP32NANO/PCB/Neowings(PCB).kicad_pcb (KiCad board)
At the start: 2 copper layers, 24.5 x 27.2 mm, 17 parts, among them J1 USB_C_Receptacle_USB2.0_16P, J3 Conn_01x17_Pin, SW1 SW_Push, SW2 SW_Push, U1 ESP32-S3-WROOM-1, U2 AMS1117-3.3

Commit message: Add files via upload
Parts:
- moved C5(1uf) 4.14 mm to (122.3, 53.9)
- moved R4(5.1k) 3.86 mm to (120.4, 76.9), turned to 0 degrees
- moved R1(10k) 3.70 mm to (120.2, 53.9)
- moved R3(5.1k)1 3.65 mm to (116.7, 76.9), turned to 180 degrees
- moved C3(22uf) 3.44 mm to (118.2, 53.9)
- moved C4(100nf) 3.06 mm to (116.1, 53.9)
- moved C6(100nf)1 1.05 mm to (116.7, 60.5), turned to 180 degrees
- moved SW1 0.26 mm to (117.9, 57.5)
Routing:
- net GND: track 4.15 -> 20.0 mm
- net +3.3V: track 17.7 -> 7.65 mm
- net Net-(J3-Pin_14): track 6.33 -> 0.00 mm
- net Net-(J3-Pin_12): track 2.72 -> 0.03 mm
- net Net-(J3-Pin_11): track 2.61 -> 0.03 mm
- net Net-(J3-Pin_10): track 2.50 -> 0.00 mm
- net Net-(J3-Pin_5): track 2.46 -> 0.00 mm
- net Net-(J3-Pin_9): track 2.39 -> 0.00 mm
- net Net-(J3-Pin_1): track 2.37 -> 0.00 mm
- net Net-(J3-Pin_4): track 2.35 -> 0.00 mm
- net Net-(J3-Pin_13): track 2.83 -> 0.66 mm
- net Net-(J3-Pin_3): track 2.24 -> 0.16 mm
- net Net-(J3-Pin_2): track 2.26 -> 0.23 mm
Other:
- board size 24.5 x 27.2 mm -> 24.5 x 27.4 mm
- board text added: "${REFERENCE}"
